Commit message: Creating launch file and modifying the urdf

File: camco_description/urdf/camco.urdf.xacro (robot description, xacro)
@@ -4,4 +4,8 @@
     <xacro:include filename="$(find kobuki_description)/urdf/kobuki.urdf.xacro" />
     <xacro:include filename="$(find turtlebot4_description)/urdf/sensors/rplidar.urdf.xacro" />
+    <xacro:include filename="$(find camco_description)/urdf/camco_platform.urdf.xacro" />
     <xacro:kobuki/>
+    <xacro:camco_platform parent_link="base_link" name="camco_platform">
+    <origin xyz="0 0 0.1356" rpy="0 0 0" />
+  </xacro:camco_platform>
 </robot>

Commit message: Fixing platform and lidar

File: camco_description/urdf/camco.urdf.xacro (robot description, xacro)
@@ -2,10 +2,16 @@
 <robot name="camco" xmlns:xacro="http://ros.org/wiki/xacro">
      <!-- Importing xacro elemnets -->
+    <xacro:include filename="$(find irobot_create_description)/urdf/common_properties.urdf.xacro"/>
     <xacro:include filename="$(find kobuki_description)/urdf/kobuki.urdf.xacro" />
     <xacro:include filename="$(find turtlebot4_description)/urdf/sensors/rplidar.urdf.xacro" />
     <xacro:include filename="$(find camco_description)/urdf/camco_platform.urdf.xacro" />
+    <xacro:property name="rplidar_z_offset"              value="${7.529272*cm2m}"/>
     <xacro:kobuki/>
     <xacro:camco_platform parent_link="base_link" name="camco_platform">
-    <origin xyz="0 0 0.1356" rpy="0 0 0" />
+    <origin xyz="0 0 0.089" rpy="0 0 0" />
   </xacro:camco_platform>
+  <xacro:rplidar name="rplidar" parent_link="lower_platform_link" gazebo="False">
+    <origin xyz="0 0 0.105"
+            rpy="0 0 ${pi/2}"/>
+  </xacro:rplidar>
 </robot>

File: camco_description/urdf/camco_platform.urdf.xacro (robot description, xacro)
@@ -35,5 +35,5 @@
     <parent link="lower_platform_link"/>
     <child link="upper_platform_link"/>
-    <origin xyz="0 0 0" rpy="0 0 0"/>
+    <origin xyz="0 0 0.06" rpy="0 0 0"/>
   </joint>
 </xacro:macro>

Commit message: Cleaning up xacro file

File: camco_description/urdf/camco.urdf.xacro (robot description, xacro)
@@ -1,17 +1,18 @@
 <?xml version="1.0"?>
 <robot name="camco" xmlns:xacro="http://ros.org/wiki/xacro">
-     <!-- Importing xacro elemnets -->
-    <xacro:include filename="$(find irobot_create_description)/urdf/common_properties.urdf.xacro"/>
+    <!-- Importing xacro elemnets -->
     <xacro:include filename="$(find kobuki_description)/urdf/kobuki.urdf.xacro" />
     <xacro:include filename="$(find turtlebot4_description)/urdf/sensors/rplidar.urdf.xacro" />
     <xacro:include filename="$(find camco_description)/urdf/camco_platform.urdf.xacro" />
-    <xacro:property name="rplidar_z_offset"              value="${7.529272*cm2m}"/>
+    <!-- Defining offsets -->
+    <xacro:property name="rplidar_z_to_platform"              value="0.105"/>
+    <xacro:property name="platform_z_to_base_link"              value="0.089"/>
+    <!-- Adding xacro elements -->
     <xacro:kobuki/>
     <xacro:camco_platform parent_link="base_link" name="camco_platform">
-    <origin xyz="0 0 0.089" rpy="0 0 0" />
-  </xacro:camco_platform>
-  <xacro:rplidar name="rplidar" parent_link="lower_platform_link" gazebo="False">
-    <origin xyz="0 0 0.105"
-            rpy="0 0 ${pi/2}"/>
-  </xacro:rplidar>
+      <origin xyz="0 0 ${platform_z_to_base_link}" rpy="0 0 0" />
+    </xacro:camco_platform>
+    <xacro:rplidar name="rplidar" parent_link="lower_platform_link" gazebo="False">
+      <origin xyz="0  0 ${rplidar_z_to_platform}" rpy="0 0 ${pi/2}"/>
+    </xacro:rplidar>
 </robot>

File: camco_description/urdf/camco_platform.urdf.xacro (robot description, xacro)
@@ -2,5 +2,5 @@
 <robot xmlns:xacro="http://ros.org/wiki/xacro">
 <xacro:macro name="camco_platform" params="name:=camco_platform parent_link:=base_link *origin">
-  <xacro:property name="mass" value="0.81144"/>
+  <xacro:property name="lower_platform_z_length" value="0.06"/>
   <xacro:property name="link_name" value="${name}_link"/>
   <xacro:property name="joint_name" value="${name}_joint"/>
@@ -35,5 +35,5 @@
     <parent link="lower_platform_link"/>
     <child link="upper_platform_link"/>
-    <origin xyz="0 0 0.06" rpy="0 0 0"/>
+    <origin xyz="0 0 ${lower_platform_z_length}" rpy="0 0 0"/>
   </joint>
 </xacro:macro>
